File: samsung16a.kicad_sch (KiCad schematic)
At the start: 0 parts

Commit message: Вибрав основний Чіп
Parts:
- added U?: STM32G431CBTx, Package_QFP:LQFP-48_7x7mm_P0.5mm, symbol MCU_ST_STM32G4:STM32G431CBTx
Connections:
- new net: U?.23 (VSS), U?.35 (VSS), U?.47 (VSS)
Changed lines of the file:
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@@
 	(generator_version "10.0")
 	(paper "A4")
+	(symbol
+		(lib_id "MCU_ST_STM32G4:STM32G431CBTx")
+		(at 152.4 102.87 0)
+		(unit 1)
+		(body_style 1)
+		(exclude_from_sim no)
+		(in_bom yes)
+		(on_board yes)
+		(in_pos_files yes)
+		(dnp no)
+		(fields_autoplaced yes)
+		(property "Reference" "U?"
+			(at 157.0833 143.51 0)
+			(show_name no)
+			(do_not_autoplace no)
+			(effects
+				(font
+					(size 1.27 1.27)
+				)
+				(justify left)
+			)
+		)
+		(property "Value" "STM32G431CBTx"
+			(at 157.0833 146.05 0)
+			(show_name no)
+			(do_not_autoplace no)
+			(effects
+				(font
+					(size 1.27 1.27)
+				)
+				(justify left)
+			)
+		)
+		(property "Footprint" "Package_QFP:LQFP-48_7x7mm_P0.5mm"
+			(at 137.16 140.97 0)
+			(hide yes)
+			(show_name no)
+			(do_not_autoplace no)
+			(effects
+				(font
+					(size 1.27 1.27)
+				)
+				(justify right)
+			)
+		)
+		(property "Datasheet" "https://www.st.com/resource/en/datasheet/stm32g431cb.pdf"
+			(at 152.4 102.87 0)
+			(hide yes)
+			(show_name no)
+			(do_not_autoplace no)
+			(effects
+				(font
+					(size 1.27 1.27)
+				)
+			)
+		)
+		(property "Description" "STMicroelectronics Arm Cortex-M4 MCU, 128KB flash, 32KB RAM, 170 MHz, 1.71-3.6V, 38 GPIO, LQFP48"
+			(at 152.4 102.87 0)
+			(hide yes)
+			(show_name no)
+			(do_not_autoplace no)
+			(effects
+				(font
+					(size 1.27 1.27)
+				)
+			)
+		)
+		(pin "4"
+		)
+		(pin "2"
+		)
+		(pin "3"
+		)
+		(pin "6"
+		)
+		(pin "7"
+		)
+		(pin "9"
+		)
+		(pin "5"
+		)
+		(pin "8"
+		)
+		(pin "1"
+		)
+		(pin "10"
+		)
+		(pin "11"
+		)
+		(pin "12"
+		)
+		(pin "13"
+		)
+		(pin "14"
+		)
+		(pin "15"
+		)
+		(pin "16"
+		)
+		(pin "20"
+		)
+		(pin "26"
+		)
+		(pin "27"
+		)
+		(pin "17"
+		)
+		(pin "22"
+		)
+		(pin "24"
+		)
+		(pin "25"
+		)
+		(pin "23"
+		)
+		(pin "18"
+		)
+		(pin "19"
+		)
+		(pin "21"
+		)
+		(pin "35"
+		)
+		(pin "28"
+		)
+		(pin "33"
+		)
+		(pin "29"
+		)
+		(pin "30"
+		)
+		(pin "31"
+		)
+		(pin "32"
+		)
+		(pin "34"
+		)
+		(pin "39"
+		)
+		(pin "36"
+		)
+		(pin "37"
+		)
+		(pin "38"
+		)
+		(pin "44"
+		)
+		(pin "43"
+		)
+		(pin "48"
+		)
+		(pin "41"
+		)
+		(pin "47"
+		)
+		(pin "42"
+		)
+		(pin "46"
+		)
+		(pin "45"
+		)
+		(pin "40"
+		)
+		(instances
+			(project "samsung16a"
+				(path "/1c8e70df-7651-4b9f-86c8-b2d78d9d3e27"
+					(reference "U?")
+					(unit 1)
+				)
+			)
+		)
+	)
 	(sheet_instances
 		(path "/"

Commit message: USB-C
Parts:
- added U?: TS3USBCA420, Package_DFN_QFN:UQFN-16_1.8x2.6mm_P0.4mm, symbol Interface_USB:TS3USBCA420
Connections:
- net at U?.15 (PA7): now also U?.11 (SBU1)
- net VSSA: now reaches U?.19 (VSSA)
- net VDDA: now reaches U?.21 (VDDA)
- net VSS: now reaches U?.23 (VSS), U?.35 (VSS), U?.47 (VSS)
- net VSS: now also U?.1 (VCC)
- net VDD: now reaches U?.24 (VDD)
- net VDD: now also U?.36 (VDD), U?.48 (VDD), U?.9 (GND)
- net at U?.30 (PA8): now also U?.10 (SBU2)
- net at U?.38 (PA14): now also U?.5 (SEL1/SCL)
- net at U?.39 (PA15): now also U?.6 (SEL0/SDA)

Commit message: добавив eepom
Parts:
- added U1: 24LC16, symbol Memory_EEPROM:24LC16
Connections:
- net at U?.3 (PC14): now also U1.6 (SCL)
- net at U?.4 (PC15): now also U1.5 (SDA)
- net at U?.42 (PB5): now also U1.4 (GND)
- net at U?.44 (PB7): now also U1.2 (A1)
Changed lines of the file:
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@@
+	(wire
+		(pts
+			(xy 129.54 92.71) (xy 134.62 92.71)
+		)
+		(stroke
+			(width 0)
+			(type default)
+		)
+	)
+	(wire
+		(pts
+			(xy 85.09 100.33) (xy 85.09 115.57)
+		)
+		(stroke
+			(width 0)
+			(type default)
+		)
+	)
+	(wire
+		(pts
+			(xy 129.54 107.95) (xy 129.54 110.49)
+		)
+		(stroke
+			(width 0)
+			(type default)
+		)
+	)
+	(wire
+		(pts
+			(xy 129.54 97.79) (xy 129.54 92.71)
+		)
+		(stroke
+			(width 0)
+			(type default)
+		)
+	)
 	(wire
 		(pts
@@
 	(wire
 		(pts
+			(xy 87.63 100.33) (xy 85.09 100.33)
+		)
+		(stroke
+			(width 0)
+			(type default)
+		)
+	)
+	(wire
+		(pts
+			(xy 129.54 110.49) (xy 134.62 110.49)
+		)
+		(stroke
+			(width 0)
+			(type default)
+		)
+	)
+	(wire
+		(pts
 			(xy 222.25 110.49) (xy 191.77 110.49)
 		)
@@
 	(wire
 		(pts
+			(xy 107.95 100.33) (xy 123.19 100.33)
+		)
+		(stroke
+			(width 0)
+			(type default)
+		)
+	)
+	(wire
+		(pts
 			(xy 170.18 107.95) (xy 222.25 107.95)
 		)
@@
 	(wire
 		(pts
+			(xy 85.09 115.57) (xy 134.62 115.57)
+		)
+		(stroke
+			(width 0)
+			(type default)
+		)
+	)
+	(wire
+		(pts
+			(xy 123.19 90.17) (xy 134.62 90.17)
+		)
+		(stroke
+			(width 0)
+			(type default)
+		)
+	)
+	(wire
+		(pts
 			(xy 180.34 92.71) (xy 180.34 87.63)
 		)
@@
 	(wire
 		(pts
+			(xy 97.79 107.95) (xy 129.54 107.95)
+		)
+		(stroke
+			(width 0)
+			(type default)
+		)
+	)
+	(wire
+		(pts
+			(xy 123.19 100.33) (xy 123.19 90.17)
+		)
+		(stroke
+			(width 0)
+			(type default)
+		)
+	)
+	(wire
+		(pts
+			(xy 107.95 97.79) (xy 129.54 97.79)
+		)
+		(stroke
+			(width 0)
+			(type default)
+		)
+	)
+	(wire
+		(pts
 			(xy 222.25 92.71) (xy 180.34 92.71)
 		)
@@
 				)
 			)
+		)
+	)
+	(symbol
+		(lib_id "Memory_EEPROM:24LC16")
+		(at 97.79 100.33 0)
+		(unit 1)
+		(body_style 1)
+		(exclude_from_sim no)
+		(in_bom yes)
+		(on_board yes)
+		(in_pos_files yes)
+		(dnp no)
+		(fields_autoplaced yes)
+		(property "Reference" "U1"
+			(at 99.9333 90.17 0)
+			(show_name no)
+			(do_not_autoplace no)
+			(effects
+				(font
+					(size 1.27 1.27)
+				)
+				(justify left)
+			)
+		)
+		(property "Value" "24LC16"
+			(at 99.9333 92.71 0)
+			(show_name no)
+			(do_not_autoplace no)
+			(effects
+				(font
+					(size 1.27 1.27)
+				)
+				(justify left)
+			)
+		)
+		(property "Footprint" ""
+			(at 97.79 100.33 0)
+			(hide yes)
+			(show_name no)
+			(do_not_autoplace no)
+			(effects
+				(font
+					(size 1.27 1.27)
+				)
+			)
+		)
+		(property "Datasheet" "http://ww1.microchip.com/downloads/en/DeviceDoc/21703d.pdf"
+			(at 97.79 100.33 0)
+			(hide yes)
+			(show_name no)
+			(do_not_autoplace no)
+			(effects
+				(font
+					(size 1.27 1.27)
+				)
+			)
+		)
+		(property "Description" "I2C Serial EEPROM, 16Kb, DIP-8/SOIC-8/TSSOP-8/DFN-8"
+			(at 97.79 100.33 0)
+			(hide yes)
+			(show_name no)
+			(do_not_autoplace no)
+			(effects
+				(font
+					(size 1.27 1.27)
+				)
+			)
+		)
+		(pin "8"
+		)
+		(pin "4"
+		)
+		(pin "2"
+		)
+		(pin "5"
+		)
+		(pin "6"
+		)
+		(pin "7"
+		)
+		(pin "1"
+		)
+		(pin "3"
+		)
+		(instances
+			(project "samsung16a"
+				(path "/1c8e70df-7651-4b9f-86c8-b2d78d9d3e27"
+					(reference "U1")
+					(unit 1)
+				)
+			)
